File: schematic_design/AT01/AT01.kicad_pcb (KiCad board)
At the start: 2 copper layers, 85 x 56 mm, 58 parts, among them J1 JST Connector, J2 Conn_01x08, J3 USB_C_Receptacle_USB2.0, J4 DC Pump Connector, J5 Solenoid Valve Connector, Q1 DMG2301L, Q2 2N7002, Q3 2N7002, SW1 SW_Push, SW2 SW_Push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

Commit message: updated FTDI board
Parts:
- added C12: 10uF, Capacitor_SMD:C_0402_1005Metric_Pad0.74x0.62mm_HandSolder, F.Cu at (182.3, 107.5)
- added C15: 0.1uF, Capacitor_SMD:C_0402_1005Metric_Pad0.74x0.62mm_HandSolder, F.Cu at (175.0, 115.7)
- added C16: 10uF, Capacitor_SMD:C_0402_1005Metric_Pad0.74x0.62mm_HandSolder, F.Cu at (181.3, 118.0)
- added C17: 0.1uF, Capacitor_SMD:C_0402_1005Metric_Pad0.74x0.62mm_HandSolder, F.Cu at (120.3, 83.7)
- added C18: 10uF, Capacitor_SMD:C_0402_1005Metric_Pad0.74x0.62mm_HandSolder, F.Cu at (123.9, 87.0)
- added C9: 10uF, Capacitor_SMD:C_0402_1005Metric_Pad0.74x0.62mm_HandSolder, F.Cu at (178.3, 102.8)
- added D10: LED, LED_THT:LED_D3.0mm, F.Cu at (185.3, 115.9)
- added D9: MBRM120LT3G, Diode_SMD:D_SOD-123F, F.Cu at (178.7, 106.9)
- added L1: 2.7u, Library:IND_R2NC_SUM, F.Cu at (184.8, 97.6)
- added Q4: FDS6375, Library:SOIC127P600X175-8N, F.Cu at (172.2, 110.7)
- added R18: 100m, Capacitor_SMD:C_0402_1005Metric_Pad0.74x0.62mm_HandSolder, F.Cu at (185.4, 107.5)
- added R19: 100K, Capacitor_SMD:C_0402_1005Metric_Pad0.74x0.62mm_HandSolder, F.Cu at (183.6, 110.9)
- added R20: 5.1K, Resistor_SMD:R_0402_1005Metric_Pad0.72x0.64mm_HandSolder, F.Cu at (143.0, 115.1)
- added U7: MCP73844T-840I/MS, Library:MSOP8_MC_MCH, F.Cu at (179.1, 113.0)
- D2: value LED -> MBRM120LT3G; footprint LED_THT:LED_D3.0mm -> Diode_SMD:D_SOD-123F
- J2: value Conn_01x08 -> Conn_01x07; footprint Connector_PinHeader_1.00mm:PinHeader_1x08_P1.00mm_Vertical -> Connector_PinHeader_1.00mm:PinHeader_1x07_P1.00mm_Vertical
- J4, J5: footprint TerminalBlock_4Ucon:TerminalBlock_4Ucon_1x02_P3.50mm_Vertical -> TerminalBlock_4Ucon:TerminalBlock_4Ucon_1x02_P3.50mm_Horizontal
- R10: value 5.1K -> 10K; footprint Resistor_SMD:R_0402_1005Metric_Pad0.72x0.64mm_HandSolder -> Capacitor_SMD:C_0402_1005Metric_Pad0.74x0.62mm_HandSolder
- R9: value 5.1K -> 61.2K
- U4: value MCP73831-2-OT -> LT1935ES5-TRPBF; footprint Package_TO_SOT_SMD:SOT-23-5 -> Library:S_5_ADI
- moved H1 91.0 mm to (185.9, 124.0)
- moved H3 90.5 mm to (109.5, 76.7)
- moved H2 84.8 mm to (178.4, 76.3)
- moved H4 80.4 mm to (109.6, 124.5)
- moved R17 51.5 mm to (122.0, 78.3), turned to 0 degrees
- moved C1 50.5 mm to (110.0, 95.2), turned to 180 degrees
- moved SW3 48.6 mm to (125.8, 73.8)
- moved C14 43.0 mm to (159.6, 99.9), turned to -90 degrees
- moved U1 41.4 mm to (115.9, 101.8), turned to 0 degrees
- moved J1 41.4 mm to (176.6, 120.7), turned to 180 degrees
- moved C11 40.9 mm to (160.0, 93.5), turned to -90 degrees
- moved C3 40.7 mm to (150.1, 90.5), turned to 180 degrees
- moved U6 40.1 mm to (161.5, 117.4), turned to 180 degrees
- moved C4 40.1 mm to (155.0, 95.5), turned to 0 degrees
- moved J4 38.7 mm to (146.4, 108.9), turned to 0 degrees
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Connections:
- C7 pad 1: GND -> VBUS
- C7 pad 2: VBAT -> GND
- D2 pad 1: GND -> Net-(D2-K)
- J2 pad 1: GND -> 3V3
- J2 pad 2: RST_SCREEN -> GND
- J2 pad 3: BL_SCREEN -> DC_SCREEN
- J2 pad 4: CS -> RST_SCREEN
- J2 pad 5: DC_SCREEN -> SCK
- J2 pad 6: SCK -> CS
- Q1 pad 2: Net-(D1-K) -> VBAT
- Q1 pad 3: VBAT -> Net-(D1-K)
- R10 pad 1: Net-(D2-A) -> Net-(U4-FB)
- R10 pad 2: Net-(U4-STAT) -> GND
- R15 pad 2: Net-(U5-IO16) -> Net-(U5-IO15)
- R16 pad 2: Net-(U5-IO21) -> Net-(U5-IO23)
- R17 pad 2: Net-(U5-IO25) -> Net-(U5-IO22)
- R9 pad 1: Net-(U4-PROG) -> Net-(D2-K)
- R9 pad 2: GND -> Net-(U4-FB)
- SW2 pad 2: Net-(U5-IO21) -> Net-(U5-IO23)
- SW3 pad 2: Net-(U5-IO25) -> Net-(U5-IO22)
- U4 pad 1: Net-(U4-STAT) -> Net-(D2-A)
- U4 pad 3: VBAT -> Net-(U4-FB)
- U4 pad 5: Net-(U4-PROG) -> VBUS
- U5 pad 10: Net-(U5-IO25) -> DC_SCREEN
- U5 pad 11: DRV_SLEEP -> RST_SCREEN
- U5 pad 12: DRV_FAULT -> unconnected-(U5-IO27-Pad12)
- U5 pad 13: SOLENOID_PIN_1 -> SCK
- U5 pad 14: MOTOR_PIN_1 -> CS
- U5 pad 16: MOTOR_PIN_2 -> MOSI
- U5 pad 23: SOLENOID_PIN_2 -> Net-(U5-IO15)
- U5 pad 26: unconnected-(U5-IO4-Pad26) -> DRV_FAULT
- U5 pad 27: Net-(U5-IO16) -> DRV_SLEEP
- U5 pad 28: unconnected-(U5-IO17-Pad28) -> SOLENOID_PIN_1
- U5 pad 29: SCK -> SOLENOID_PIN_2
- U5 pad 30: MOSI -> MOTOR_PIN_1
- U5 pad 31: unconnected-(U5-IO19-Pad31) -> MOTOR_PIN_2
- U5 pad 33: Net-(U5-IO21) -> unconnected-(U5-IO21-Pad33)
- U5 pad 36: SCL -> Net-(U5-IO22)
- U5 pad 37: SDA -> Net-(U5-IO23)
- U5 pad 6: RST_SCREEN -> SCL
- U5 pad 7: BL_SCREEN -> SDA
- U5 pad 8: CS -> unconnected-(U5-IO32-Pad8)
- U5 pad 9: DC_SCREEN -> unconnected-(U5-IO33-Pad9)
Routing:
- net Net-(U5-SENSOR_VP): track 16.8 -> 52.5 mm, vias 0 -> 2
- net Net-(U5-IO25): track 31.3 -> 0.00 mm, vias 2 -> 0
- net VBAT: track 86.3 -> 55.6 mm, vias 4 -> 2
- net Net-(U5-IO21): track 25.8 -> 0.00 mm, vias 1 -> 0
- net Net-(U5-IO22): track 0.00 -> 24.8 mm
- net Net-(D10-A): track 0.00 -> 20.4 mm
- net SCK: track 23.9 -> 3.66 mm, vias 2 -> 0
- net GPIO0: track 13.9 -> 33.0 mm, vias 0 -> 2
- net SOLENOID_PIN_2: track 27.1 -> 10.9 mm
- net Net-(U5-IO23): track 0.00 -> 15.6 mm
- net Net-(U7-SENSE): track 0.00 -> 15.6 mm, vias 0 -> 3
- net Net-(J4-Pin_2): track 24.1 -> 9.71 mm, vias 2 -> 0
- net Net-(U7-DRV): track 0.00 -> 14.1 mm, vias 0 -> 2
- net EN: track 59.5 -> 45.7 mm
- net MOSI: track 22.6 -> 9.62 mm, vias 2 -> 0
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Other:
- board text added: "DH^{3} TOURNIQUET SYSTEM"
- board text removed: "AT01"
- board text removed: "DH^{3} TOURNIQUET Rev 1.0"
- board text removed: "Designed by: Diana Temelkos Hassan Khan Haashim Shahzada Sayeed Hasan"
