File: schematic_design/AT01/AT01_Lipo.kicad_sch (KiCad schematic)
At the start: 0 parts

Commit message: adding design recommendations from call with Yi
Parts:
- added C1: 4.7uF, Capacitor_SMD:C_0402_1005Metric_Pad0.74x0.62mm_HandSolder, symbol Device:C
- added C2, C3: 10uF, Capacitor_SMD:C_0402_1005Metric_Pad0.74x0.62mm_HandSolder, symbol Device:C
- added C4: 0.1uF, Capacitor_SMD:C_0402_1005Metric_Pad0.74x0.62mm_HandSolder, symbol Device:C_Small
- added C5: 10uF, Capacitor_SMD:C_0402_1005Metric_Pad0.74x0.62mm_HandSolder, symbol Device:C_Small
- added D1, D2: MBRM120LT3G, Diode_SMD:D_SOD-123F, symbol Diode:MBR1020VL
- added D3: LED, LED_THT:LED_D3.0mm, symbol Device:LED
- added L1: 2.7u, Library:IND_R2NC_SUM, symbol Device:L
- added Q1: FDS6375, Library:SOIC127P600X175-8N, symbol FDS6375:FDS6375
- added R1: 61.2K, Resistor_SMD:R_0402_1005Metric_Pad0.72x0.64mm_HandSolder, symbol Device:R
- added R2: 10K, Capacitor_SMD:C_0402_1005Metric_Pad0.74x0.62mm_HandSolder, symbol Device:R
- added R3: 100m, Capacitor_SMD:C_0402_1005Metric_Pad0.74x0.62mm_HandSolder, symbol Device:R
- added R4: 100K, Capacitor_SMD:C_0402_1005Metric_Pad0.74x0.62mm_HandSolder, symbol Device:R
- added U1: LT1935ES5-TRPBF, S_5_ADI, symbol 2023-10-27_15-39-09:LT1935ES5-TRPBF
- added U2: MCP73844T-840I/MS, MSOP8_MC_MCH, symbol 2023-10-27_15-39-09:MCP73844T-840I_MS
Connections:
- new net: C2.1, D1.1 (K), D2.2 (A), R1.1
- new net: C4.1, U2.5 (TIMER)
- new net: D3.1 (K), U2.3 (STAT1)
- new net: C3.1, D2.1 (K), D3.2 (A), R3.1, R4.1, U2.2 (VDD)
- new net: R4.2, U2.4 (EN)
- new net: R1.2, R2.1, U1.3 (FB)
- new net: Q1.1, R3.2, U2.1 (SENSE)
- new net: D1.2 (A), L1.2, U1.1 (SW)
- new net: Q1.4, U2.8 (DRV)
- new net GND: C1.2, C2.2, C3.2, C4.2, C5.2, R2.2, U1.2 (GND), U2.6 (VSS)
- new net VBAT: C5.1, Q1.5, U2.7 (VBAT)
- new net VBUS: C1.1, L1.1, U1.4 (*SHDN), U1.5 (VIN)
Other:
- note added: "9V"
- note added: "LIPO CHARGING CIRCUIT"
