File: schematic_design/AT01/AT01_no_ftdi.kicad_sch (KiCad schematic)
At the start: 49 parts, among them J1 JST Connector, J2 USB_C_Receptacle_USB2.0, J3 Conn_01x08, J4 Solenoid Valve Connector, J5 DC Pump Connector, J6 PPG Sensor Input, K1 TLP4590ATP1_F, SW1 SW_Push, SW2 SW_Push, SW3 SW_Push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

Commit message: updating load sharing circuit
Parts:
- removed J2: USB_C_Receptacle_USB2.0, Library:GCT_USB4085-GF-A_REVB, symbol 2023-10-27_15-39-09:USB4085-GF-A_REVB
- added J2: USB4125-GF-A-0190, CONN6_125-GF-A-0190_GCT, symbol 2023-10-27_15-39-09:USB4125-GF-A-0190
- added J7: RX/TX Breakout, Connector_PinHeader_2.54mm:PinHeader_1x02_P2.54mm_Vertical, symbol Connector_Generic:Conn_01x02
Connections:
- net GND: now also J2.1 (GND), J2.6 (GND)
- net VBUS: now also J2.2 (VBUS), J2.5 (VBUS)
- net VCC: now reaches C5.1, K1.2, K1.4, U4.3 (VI)
- net VCC: now also C10.2, C12.1, C9.2, R4.2, U5.12 (VM)
- net at U6.13 (IO19): now also R11.1
- net at U6.14 (IO20): now also R10.2
- net at U6.36 (RXD0): now also J7.1 (Pin_1); no longer R10.2
- net at U6.37 (TXD0): now also J7.2 (Pin_2); no longer R11.1
- net at R13.1: now also J2.3 (CC1)
- net at R14.1: now also J2.4 (CC2)
- removed net VBAT: C10.2, C12.1, C9.2, D2.1 (K), D2.2 (A), J1.1 (Pin_1), K1.1, R4.2, U5.12 (VM)
- new net: D2.1 (K), K1.1
- new net: D2.2 (A), J1.1 (Pin_1)
- no-connect marks 27 -> 19
Other:
- note removed: "Change Q1 to SSR TLP4590A(TP1,F)"
- note removed: "LDO reaches 220 C, consider buck converter or TO-220 package"
- note removed: "May or may not need current control resistor for AISEN, BISEN"
- note removed: "Notes: Add a P&ID Diagram -> Process and Instrumentation Diagram Industry standards for locking (JST and stuff) ESD blows up the gate or the fuse, you want to spec this diode, less than or equal to operating voltage working voltage -> priority ADC will not properly track battery voltage (accuracy is very sus) multimeter is x4 more accurate breakdown voltage is less than abs max pick a uni-directi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"
- moved on the sheet: C17, C18, C20, C5, C7, D2, D4, D5, J1, J3, K1, R10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

Commit message: Rev3.0 board commits
Parts:
- removed J2: USB4125-GF-A-0190, CONN6_125-GF-A-0190_GCT, symbol 2023-10-27_15-39-09:USB4125-GF-A-0190
- added J2: USB4125-GF-A-0190_REVA2, Library:GCT_USB4125-GF-A-0190_REVA2, symbol 2023-10-27_15-39-09:USB4125-GF-A-0190_REVA2
Connections:
- net GND: now also J2.A12 (GND), J2.B12 (GND__1), J2.S1 (SHIELD), J2.S2 (SHIELD__1), J2.S3 (SHIELD__2), J2.S4 (SHIELD__3)
- net VBUS: now also J2.A9 (VBUS), J2.B9 (VBUS__1)
- net at R13.1: now also J2.A5 (CC1)
- net at R14.1: now also J2.B5 (CC2)
Other:
- moved on the sheet: R13, R14
